File: integrated_circuits.kicad_sch (KiCad schematic)
At the start: 0 parts

Commit message: Add diode arrays
Parts:
- added U? (x13): S16-4148, symbol Arrays:S16-4148
- added U?: ESP32-WROOM-32D, RF_Module:ESP32-WROOM-32, symbol RF_Module:ESP32-WROOM-32D
Connections:
- new net GND: U?.1 (GND), U?.15 (GND), U?.38 (GND), U?.39 (GND)
- new net R0C00: U?.16
- new net R0C01: U?.15
- new net R0C02: U?.14
- new net R0C03: U?.13
- new net R0C04: U?.12
- new net R0C05: U?.11
- new net R0C06: U?.10
- new net R0C07: U?.9
- new net R0C08: U?.16
- new net R0C09: U?.15
- new net R0C10: U?.14
- new net R0C11: U?.13
- new net R0C12: U?.12
- new net R1C00: U?.11
- new net R1C01: U?.10
- new net R1C02: U?.9
- new net R1C03: U?.16
- new net R1C04: U?.15
- new net R1C05: U?.14
- new net R1C06: U?.13
- new net R1C07: U?.12
- new net R1C08: U?.11
- new net R1C09: U?.10
- new net R1C10: U?.9
- new net R1C11: U?.16
- new net R1C12: U?.15
- new net R2C00: U?.14
- new net R2C01: U?.13
- new net R2C02: U?.12
- new net R2C03: U?.11
- new net R2C04: U?.10
- new net R2C05: U?.9
- new net R2C06: U?.16
- new net R2C07: U?.15
- new net R2C08: U?.14
- new net R2C09: U?.13
- new net R2C10: U?.12
- new net R2C11: U?.11
- new net R2C12: U?.10
- new net R3C00: U?.9
- new net R3C01: U?.16
- new net R3C02: U?.15
- new net R3C03: U?.14
- new net R3C04: U?.13
- new net R3C05: U?.12
- new net R3C06: U?.11
- new net R3C07: U?.10
- new net R3C08: U?.9
- new net R3C09: U?.16
- new net R3C10: U?.15
- new net R3C11: U?.14
- new net R3C12: U?.13
- new net R4C00: U?.12
- new net R4C01: U?.11
- new net R4C02: U?.10
- new net R4C03: U?.9
- new net R4C04: U?.16
- new net R4C05: U?.15
- new net R4C06: U?.14
- new net R4C07: U?.13
- new net R4C08: U?.12
- new net R4C09: U?.11
- new net R4C10: U?.10
- new net R4C11: U?.9
- new net R4C12: U?.16
- new net R5C00: U?.15
- new net R5C01: U?.14
- new net R5C02: U?.13
- new net R5C03: U?.12
- new net R5C04: U?.11
- new net R5C05: U?.10
- new net R5C06: U?.9
- new net R5C07: U?.16
- new net R5C08: U?.15
- new net R5C09: U?.14
- new net R5C10: U?.13
- new net R5C11: U?.12
- new net R5C12: U?.11
- new net R6C00: U?.10
- new net R6C01: U?.9
- new net R6C02: U?.16
- new net R6C03: U?.15
- new net R6C04: U?.14
- new net R6C05: U?.13
- new net R6C06: U?.12
- new net R6C07: U?.11
- new net R6C08: U?.10
- new net R6C09: U?.9
- new net R6C10: U?.16
- new net R6C11: U?.15
- new net R6C12: U?.14
- new net R7C00: U?.13
- new net R7C01: U?.12
- new net R7C02: U?.11
- new net R7C03: U?.10
- new net R7C04: U?.9
- new net R7C05: U?.16
- new net R7C06: U?.15
- new net R7C07: U?.14
- new net R7C08: U?.13
- new net R7C09: U?.12
- new net R7C10: U?.11
- new net R7C11: U?.10
- new net R7C12: U?.9
- new net VDD: U?.2 (VDD)
