File: keyboard.kicad_sch (KiCad schematic)
At the start: 104 parts, among them SW1 SW_DIP_x01, SW10 SW_DIP_x01, SW100 SW_DIP_x01, SW101 SW_DIP_x01, SW102 SW_DIP_x01, SW103 SW_DIP_x01, SW104 SW_DIP_x01, SW11 SW_DIP_x01, SW12 SW_DIP_x01, SW13 SW_DIP_x01, SW14 SW_DIP_x01, SW15 SW_DIP_x01, SW16 SW_DIP_x01, SW17 SW_DIP_x01, SW18 SW_DIP_x01, SW19 SW_DIP_x01, SW2 SW_DIP_x01, SW20 SW_DIP_x01, SW21 SW_DIP_x01, SW22 SW_DIP_x01, SW23 SW_DIP_x01, SW24 SW_DIP_x01, SW25 SW_DIP_x01, SW26 SW_DIP_x01, SW27 SW_DIP_x01, SW28 SW_DIP_x01, SW29 SW_DIP_x01, SW3 SW_DIP_x01, SW30 SW_DIP_x01, SW31 SW_DIP_x01, SW32 SW_DIP_x01, SW33 SW_DIP_x01, SW34 SW_DIP_x01, SW35 SW_DIP_x01, SW36 SW_DIP_x01, SW37 SW_DIP_x01, SW38 SW_DIP_x01, SW39 SW_DIP_x01, SW4 SW_DIP_x01, SW40 SW_DIP_x01, SW41 SW_DIP_x01, SW42 SW_DIP_x01, SW43 SW_DIP_x01, SW44 SW_DIP_x01, SW45 SW_DIP_x01, SW46 SW_DIP_x01, SW47 SW_DIP_x01, SW48 SW_DIP_x01, SW49 SW_DIP_x01, SW5 SW_DIP_x01, SW50 SW_DIP_x01, SW51 SW_DIP_x01, SW52 SW_DIP_x01, SW53 SW_DIP_x01, SW54 SW_DIP_x01, SW55 SW_DIP_x01, SW56 SW_DIP_x01, SW57 SW_DIP_x01, SW58 SW_DIP_x01, SW59 SW_DIP_x01, SW6 SW_DIP_x01, SW60 SW_DIP_x01, SW61 SW_DIP_x01, SW62 SW_DIP_x01, SW63 SW_DIP_x01, SW64 SW_DIP_x01, SW65 SW_DIP_x01, SW66 SW_DIP_x01, SW67 SW_DIP_x01, SW68 SW_DIP_x01, SW69 SW_DIP_x01, SW7 SW_DIP_x01, SW70 SW_DIP_x01, SW71 SW_DIP_x01, SW72 SW_DIP_x01, SW73 SW_DIP_x01, SW74 SW_DIP_x01, SW75 SW_DIP_x01, SW76 SW_DIP_x01, SW77 SW_DIP_x01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

Commit message: Roughly place LEDs. Add decoupling caps to schematic for LEDs.
Parts:
- SW1, SW10, SW100, SW101, SW102, SW103, SW104, SW11, SW12, SW13, SW14, SW15, SW16, SW17, SW18, SW19, SW2, SW20, SW21, SW22, SW23, SW24, SW25, SW26, SW27, SW28, SW29, SW3, SW30, SW31, SW32, SW33, SW34, SW35, SW36, SW37, SW38, SW39, SW4, SW40, SW41, SW42, SW43, SW44, SW45, SW46, SW47, SW48, SW49, SW5, SW50, SW51, SW52, SW53, SW54, SW55, SW56, SW57, SW58, SW59, SW6, SW60, SW61, SW62, SW63, SW64, SW65, SW66, SW67, SW68, SW69, SW7, SW70, SW71, SW72, SW73, SW74, SW75, SW76, SW77, SW78, SW79, SW8, SW80, SW81, SW82, SW83, SW84, SW85, SW86, SW87, SW88, SW89, SW9, SW90, SW91, SW92, SW93, SW94, SW95, SW96, SW97, SW98, SW99: footprint keyswitches:Kailh_socket_MX_optional_reversible -> Switch_Keyboard_Hotswap_Kailh:SW_Hotswap_Kailh_MX
